File: Transistor Tester.brd (EAGLE design)
At the start: 160 x 100 mm, 23 parts, among them Q1 BC547

Commit message: Time to start routing
Parts:
- moved C8 1.27 mm to (3.81, 35.6)
- moved C7 1.27 mm to (3.81, 29.2)
- moved MCU 1.27 mm to (57.1, 19.1)
- moved Q1 1.27 mm to (66.0, 31.8), turned to 0 degrees
Other:
- board size 160 x 100 mm -> 82.5 x 39.4 mm
- board text added: "Nathan Campos, 2013"
- board text added: "Transistor Tester"

Commit message: DONE
Parts:
- turned R1 to 0 degrees
Routing:
- net VCC: track 0.00 -> 187.9 mm, vias 0 -> 2
- net N$5: track 0.00 -> 69.8 mm, vias 0 -> 1
- net N$10: track 0.00 -> 43.8 mm, vias 0 -> 2
- net RS: track 0.00 -> 43.2 mm
- net DB7: track 0.00 -> 35.9 mm
- net BT_TEST: track 0.00 -> 35.6 mm
- net N$2: track 0.00 -> 33.1 mm
- net N$6: track 0.00 -> 32.0 mm
- net DB5: track 0.00 -> 31.2 mm
- net LCD_EN: track 0.00 -> 30.5 mm
- net N$1: track 0.00 -> 30.3 mm
- net C: track 25.5 -> 55.3 mm, vias 2 -> 3
- net N$3: track 0.00 -> 29.8 mm
- net RESET: track 0.00 -> 29.3 mm, vias 0 -> 1
- net AR: track 0.00 -> 27.5 mm
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- added copper zone on layer 1, net GND
- added copper zone on layer 16, net GND
Other:
- board text added: "CR2032"
