File: Transistor Tester.sch (EAGLE design)
At the start: 4 parts

Commit message: Added a bunch of stuff
Parts:
- added 7805: 7805TV, linear:7805TV
- added BAT1, BAT2: 20mm coincell, SparkFun-Electromechanical:BATTERY20MM_4LEGS
- added C2: 0.1uF, rcl:C-EU025-025X050
- added C7: 2.2uF, rcl:CPOL-EUE2.5-6
- added C8: 10uF, rcl:CPOL-EUE2.5-6
- added C9: 0.1uF, rcl:C-EU050-025X075
- added IC1: MEGA8-P, atmel:MEGA8-P
- added LCD: LCD-16X28X2, SparkFun-Displays:LCD-16X28X2
- added Q1: BC547, transistor-npn:BC547
- added R4, R5: 10kΩ, rcl:R-EU_0207/10
- added SMD_PROBE: BC817-25SMD, transistor-npn:BC817-25SMD
- added VO: 10kΩ, bourns:3362H
- renumbered JP1 to PTH_PROBE
Connections:
- new net BKL_CTRL: R4.1
- new net DB4: LCD.DB4
- new net DB5: LCD.DB5
- new net DB6: LCD.DB6
- new net DB7: LCD.DB7
- new net GND: 7805.GND, BAT1.-, C2.1, C7.-, C8.-, C9.1, IC1.GND, IC1.GND@1, LCD.R/W, LCD.VSS, Q1.E, VO.3
- new net LCD_EN: LCD.E
- new net N$1: BAT1.+, BAT2.-
- new net N$10: LCD.VO, VO.2
- new net N$11: IC1.PB1(OC1A)
- new net N$12: IC1.PB0(ICP)
- new net N$2: C2.2, IC1.AREF
- new net N$3: LCD.K, Q1.C
- new net N$4: Q1.B, R4.2
- new net N$5: IC1.PB5(SCK)
- new net N$6: IC1.PB4(MISO)
- new net N$7: 7805.VI, BAT2.+, C7.+
- new net N$8: IC1.PB3(MOSI/OC2)
- new net N$9: IC1.PB2(SS/OC1B)
- new net RESET: IC1.PC6(/RESET), R5.2
- new net RS: LCD.RS
- new net VCC: 7805.VO, C8.+, C9.2, IC1.AVCC, IC1.VCC@1, LCD.A, LCD.VDD, R5.1, VO.1
- net A: now also IC1.PD0(RXD), SMD_PROBE.B
- net AR: now also IC1.PD5(T1)
- net B: now also IC1.PD1(TXD), SMD_PROBE.C
- net BR: now also IC1.PD6(AIN0)
- net C: now also IC1.PD4(XCK/T0), SMD_PROBE.E
- net CR: now also IC1.PD7(AIN1)
Other:
- note added: "Check if the 7805 can regulate from 6V!!!!"
- note added: "Create one of those soft power ON circuits where the MCU keeps the input transistor ON and auto power off by killing it"
- note added: "Maybe measure the voltage drop across the transsitor, etc. Also, add a voltage ref to make the readings more accurate."
- note added: "Or maybe use a switch and a "Test" button"
- note added: "Test if the battery holder fits the footprint"

Commit message: Made a bunch of changes and started working in the board layout
Parts:
- added ON: (no value), led:LED3MM
- added R6: 1kΩ, rcl:R-EU_0207/10
- added SBKL, STEST: DTS-3, switch-tact:DTS-3
- added SPWR: (no value), SparkFun-Electromechanical:SWITCH-SPDTPTH
- renumbered IC1 to MCU
Connections:
- removed net N$11: MCU.PB1(OC1A)
- removed net N$12: MCU.PB0(ICP)
- removed net N$8: MCU.PB3(MOSI/OC2)
- removed net N$9: MCU.PB2(SS/OC1B)
- new net BT_BKL: MCU.PD3(INT1), SBKL.2
- new net BT_TEST: MCU.PD2(INT0), STEST.2
- net A: now also MCU.PD4(XCK/T0); no longer MCU.PD0(RXD)
- net AR: now also MCU.PC0(ADC0); no longer MCU.PD5(T1)
- net B: now also MCU.PD5(T1); no longer MCU.PD1(TXD)
- net BKL_CTRL: now also MCU.PC3(ADC3)
- net BR: now also MCU.PC1(ADC1); no longer MCU.PD6(AIN0)
- net C: now also MCU.PD6(AIN0); no longer MCU.PD4(XCK/T0)
- net CR: now also MCU.PC2(ADC2); no longer MCU.PD7(AIN1)
- net DB4: now also MCU.PB2(SS/OC1B)
- net DB5: now also MCU.PB3(MOSI/OC2)
- net DB6: now also MCU.PB4(MISO)
- net DB7: now also MCU.PB5(SCK)
- net GND: now also R6.1, SBKL.1, STEST.1
- net LCD_EN: now also MCU.PB1(OC1A)
- net N$5: now also ON.C, R6.2; no longer MCU.PB5(SCK)
- net N$6: now also BAT2.+, SPWR.P; no longer MCU.PB4(MISO)
- net N$7: now also SPWR.O; no longer BAT2.+
- net RS: now also MCU.PB0(ICP)
- net VCC: now also ON.A
Other:
- note added: "Cut a 4 pin female header or use one of those machined pin headers"
- note added: "Test if these buttons match with the ones I bought"
- note added: "Use a thin square LED horizontally"
- note removed: "Create one of those soft power ON circuits where the MCU keeps the input transistor ON and auto power off by killing it"
- note removed: "Or maybe use a switch and a "Test" button"
- moved on the sheet: BAT1, BAT2

Commit message: DONE
Other:
- note removed: "Maybe measure the voltage drop across the transsitor, etc. Also, add a voltage ref to make the readings more accurate."
Changed lines of the file:
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@@
 <sheet>
 <plain>
-<text x="259.08" y="20.32" size="1.778" layer="91">Maybe measure the
-voltage drop across
-the transsitor, etc.
-Also, add a voltage ref
-to make the readings
-more accurate.</text>
 <text x="129.54" y="-38.1" size="1.778" layer="91">Test if the battery
 holder fits the
