File: Rev B.brd (EAGLE design)
At the start: 82.5 x 39.4 mm, 23 parts, among them Q1 BC547

Commit message: Rev B schematic
Parts:
- removed BAT1, BAT2: 20mm coincell, SparkFun-Electromechanical:BATTCON_20MM_4LEGS
- removed SPWR: (no value), SparkFun-Electromechanical:SWITCH-SPDT
- added VIN: M02JST-PTH-2, SparkFun-Connectors:JST-2-PTH
Connections:
- removed net N$1: BAT1.1, BAT2.2
- removed net N$6: BAT2.1, SPWR.2
- net A: now also MCU.23; no longer MCU.6
- net AR: now also MCU.6; no longer MCU.23
- net B: now also MCU.24; no longer MCU.11
- net BR: now also MCU.11; no longer MCU.24
- net C: now also MCU.25; no longer MCU.12
- net CR: now also MCU.12; no longer MCU.25
- net GND: now also VIN.1; no longer BAT1.2
- net N$7: now also VIN.2; no longer SPWR.1
Routing:
- net N$6: track 32.0 -> 0.00 mm
- net N$1: track 30.3 -> 0.00 mm
- net A: track 42.1 -> 37.0 mm
- net CR: track 16.3 -> 12.5 mm
- net BR: track 26.5 -> 22.6 mm
- net B: track 42.5 -> 38.7 mm
- net AR: track 27.5 -> 23.7 mm
- net N$7: track 23.7 -> 20.1 mm
- net C: track 55.3 -> 54.0 mm
